Commit message: adding model to myslam-launch

File: myslam_sim_resources/robot/myslam_robot.urdf (robot description, URDF)
Before this commit: robot myfirst, 3 links, 2 joints
Links:
- link logical_camera_link: geometry collision box size=0.2 0.2 0.2; visual box size=0.2 0.2 0.2

Commit message: restructuring stacks

File: myslam_sim_resources/robot/myslam_robot.urdf (robot description, URDF)
Before this commit: robot myfirst, 3 links, 2 joints
Links:
- link base_link: geometry visual box size=.4 .2 .1
- link camera_link: geometry collision box size=.1 .1 .1; visual box size=.1 .1 .1
- link logical_camera_link: geometry collision box size=0.1 0.1 0.1; visual box size=0.1 0.1 0.1
