Commit message: adding myslam_system

File: myslam_sim_resources/robot/pioneer3at.urdf (robot description, URDF)
Before this commit: robot pioneer3at, 18 links, 17 joints
Links:
- link back_sonar: geometry collision box size=0 0 0; visual mesh filename=package://myslam_sim_resources/meshes/p3at_meshes/back_sona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
- link base_link: geometry collision mesh filename=package://myslam_sim_resources/meshes/p3at_meshes/chassis.s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; visual mesh filename=package://myslam_sim_resources/meshes/p3at_meshes/chassis.s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
- link front_sonar: geometry collision box size=0 0 0; visual mesh filename=package://myslam_sim_resources/meshes/p3at_meshes/front_son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
- link p3at_back_left_axle: geometry collision mesh filename=package://myslam_sim_resources/meshes/p3at_meshes/axle.stl; visual mesh filename=package://myslam_sim_resources/meshes/p3at_meshes/axle.stl
- link p3at_back_left_hub: geometry collision mesh filename=package://myslam_sim_resources/meshes/p3at_meshes/left_hubc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; visual mesh filename=package://myslam_sim_resources/meshes/p3at_meshes/left_hubc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
- link p3at_back_left_wheel: geometry collision cylinder length=0.075 radius=0.111; visual mesh filename=package://myslam_sim_resources/meshes/p3at_meshes/wheel.stl
- link p3at_back_right_axle: geometry collision mesh filename=package://myslam_sim_resources/meshes/p3at_meshes/axle.stl; visual mesh filename=package://myslam_sim_resources/meshes/p3at_meshes/axle.stl
- link p3at_back_right_hub: geometry collision mesh filename=package://myslam_sim_resources/meshes/p3at_meshes/right_hub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; visual mesh filename=package://myslam_sim_resources/meshes/p3at_meshes/right_hub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
- link p3at_back_right_wheel: geometry collision cylinder length=0.075 radius=0.111; visual mesh filename=package://myslam_sim_resources/meshes/p3at_meshes/wheel.stl
- link p3at_front_left_axle: geometry collision box size=0 0 0; visual mesh filename=package://myslam_sim_resources/meshes/p3at_meshes/axle.stl
- link p3at_front_left_hub: geometry collision box size=0 0 0; visual mesh filename=package://myslam_sim_resources/meshes/p3at_meshes/left_hubc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
- link p3at_front_left_wheel: geometry collision cylinder length=0.075 radius=0.111; visual mesh filename=package://myslam_sim_resources/meshes/p3at_meshes/wheel.stl
- link p3at_front_right_axle: geometry collision box size=0 0 0; visual mesh filename=package://myslam_sim_resources/meshes/p3at_meshes/axle.stl
- link p3at_front_right_hub: geometry collision box size=0 0 0; visual mesh filename=package://myslam_sim_resources/meshes/p3at_meshes/right_hub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
- link p3at_front_right_wheel: geometry collision cylinder length=0.075 radius=0.111; visual mesh filename=package://myslam_sim_resources/meshes/p3at_meshes/wheel.stl
- link top_plate: geometry collision box size=0 0 0; visual mesh filename=package://myslam_sim_resources/meshes/p3at_meshes/top.stl

Commit message: refactoring + simulation with gazebo + display objects with rviz

File: myslam_sim_resources/robot/pioneer3at.urdf (robot description, URDF)
Before this commit: robot pioneer3at, 18 links, 17 joints
Links:
- link base_link: mass 60.0 -> 100.0

Commit message: RC 1

File: myslam_sim_resources/robot/pioneer3at.urdf (robot description, URDF)
Before this commit: robot pioneer3at, 18 links, 17 joints
Links:
- added link hokuyo_link, mass 1e-5; collision box size=0.1 0.1 0.1; visual mesh filename=package://myslam_sim_resources/models/hokuyo/meshes/hokuyo.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
Joints:
- added joint hokuyo_joint: type fixed, parent base_link, child hokuyo_link, origin xyz=0 0 0.474 rpy=0 0 0, axis 0 1 0
